File: Circuit/GarageDoorController/GarageDoorController.kicad_pcb (KiCad board)
At the start: 2 copper layers, 71.5 x 50.6 mm, 27 parts, among them J3 JST PH 2-pin, J4 JST PH 4-pin, U1 XIAO-ESP32-C3-DIP, U3 TLP222A, U4 PC817, U5 R-78E5.0-0.5

Commit message: Rev 2 PCB all references to FLASH changed LAMP + Controller housing
Connections:
- net /Opener control/FLASH renamed /Opener control/LAMP
Other:
- board text removed: "GarageDoor Controller Rev 1"
Changed lines of the file:
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@@
 			(layers "*.Cu" "*.Mask")
 			(remove_unused_layers no)
-			(net "/Opener control/FLASH")
+			(net "/Opener control/LAMP")
 			(pintype "passive")
 		)
@@
 			(layers "*.Cu" "*.Mask")
 			(remove_unused_layers no)
-			(net "/Opener control/FLASH")
+			(net "/Opener control/LAMP")
 			(pinfunction "Pin_3_3")
 			(pintype "passive")
@@
 		(layer "Edge.Cuts")
 	)
-	(gr_text "GarageDoor Controller Rev 1"
-		(at 125.17 125.6 0)
-		(layer "F.SilkS")
-		(effects
-			(font
-				(size 1 1)
-				(thickness 0.1)
-			)
-			(justify left bottom)
-		)
+	(segment
+		(start 124.42132 97.62132)
+		(end 124.42132 87.23868)
+		(width 0.2)
+		(layer "F.Cu")
+		(net "+3V3")
+	)
+	(segment
+		(start 127.2 86.04132)
+		(end 138.04132 86.04132)
+		(width 0.3)
+		(layer "F.Cu")
+		(net "+3V3")
+	)
+	(segment
+		(start 125.61868 86.04132)
+		(end 127.2 86.04132)
+		(width 0.2)
+		(layer "F.Cu")
+		(net "+3V3")
+	)
+	(segment
+		(start 124.42132 87.23868)
+		(end 125.61868 86.04132)
+		(width 0.2)
+		(layer "F.Cu")
+		(net "+3V3")
+	)
+	(segment
+		(start 130.41132 103.61132)
+		(end 124.42132 97.62132)
+		(width 0.2)
+		(layer "F.Cu")
+		(net "+3V3")
+	)
+	(segment
+		(start 138.04132 86.04132)
+		(end 140 88)
+		(width 0.3)
+		(layer "F.Cu")
+		(net "+3V3")
+	)
+	(segment
+		(start 127.84868 103.61132)
+		(end 118.95868 112.50132)
+		(width 0.2)
+		(layer "B.Cu")
+		(net "+3V3")
+	)
+	(segment
+		(start 130.41132 103.61132)
+		(end 127.84868 103.61132)
+		(width 0.2)
+		(layer "B.Cu")
+		(net "+3V3")
+	)
+	(segment
+		(start 118.95868 112.50132)
+		(end 116.51132 112.50132)
+		(width 0.2)
+		(layer "B.Cu")
+		(net "+3V3")
+	)
+	(segment
+		(start 111.96 88.58132)
+		(end 116.69132 88.58132)
+		(width 0.2)
+		(layer "B.Cu")
+		(net "OPENER_MOVING")
+	)
+	(segment
+		(start 116.69132 88.58132)
+		(end 120.55 92.44)
+		(width 0.2)
+		(layer "B.Cu")
+		(net "OPENER_MOVING")
+	)
+	(segment
+		(start 140 98.16)
+		(end 138.3 99.86)
+		(width 0.2)
+		(layer "B.Cu")
+		(net "OPENER_MOVING")
+	)
+	(segment
+		(start 129.97 99.64)
+		(end 134.33 104)
+		(width 0.2)
+		(layer "B.Cu")
+		(net "OPENER_MOVING")
+	)
+	(segment
+		(start 120.55 99.64)
+		(end 129.97 99.64)
+		(width 0.2)
+		(layer "B.Cu")
+		(net "OPENER_MOVING")
+	)
+	(segment
+		(start 138.3 99.86)
+		(end 138.3 104)
+		(width 0.2)
+		(layer "B.Cu")
+		(net "OPENER_MOVING")
+	)
+	(segment
+		(start 134.33 104)
+		(end 140 104)
+		(width 0.2)
+		(layer "B.Cu")
+		(net "OPENER_MOVING")
+	)
+	(segment
+		(start 120.55 92.44)
+		(end 120.55 99.64)
+		(width 0.2)
+		(layer "B.Cu")
+		(net "OPENER_MOVING")
 	)
 	(segment
@@
 	)
 	(segment
-		(start 152.5 114.16)
-		(end 153.2 114.16)
-		(width 0.2)
-		(layer "B.Cu")
-		(net "/Opener control/FLASH")
-	)
-	(segment
-		(start 153.2 114.16)
-		(end 155.5 116.46)
-		(width 0.2)
-		(layer "B.Cu")
-		(net "/Opener control/FLASH")
-	)
-	(segment
-		(start 155.5 116.46)
-		(end 155.5 124.44)
-		(width 0.2)
-		(layer "B.Cu")
-		(net "/Opener control/FLASH")
-	)
-	(segment
 		(start 160.17 122.3)
 		(end 163.5 122.3)
@@
 	)
 	(segment
-		(start 124.42132 97.62132)
-		(end 124.42132 87.23868)
-		(width 0.2)
-		(layer "F.Cu")
-		(net "+3V3")
-	)
-	(segment
-		(start 127.2 86.04132)
-		(end 138.04132 86.04132)
-		(width 0.3)
-		(layer "F.Cu")
-		(net "+3V3")
-	)
-	(segment
-		(start 125.61868 86.04132)
-		(end 127.2 86.04132)
-		(width 0.2)
-		(layer "F.Cu")
-		(net "+3V3")
-	)
-	(segment
-		(start 124.42132 87.23868)
-		(end 125.61868 86.04132)
-		(width 0.2)
-		(layer "F.Cu")
-		(net "+3V3")
-	)
-	(segment
-		(start 130.41132 103.61132)
-		(end 124.42132 97.62132)
-		(width 0.2)
-		(layer "F.Cu")
-		(net "+3V3")
-	)
-	(segment
-		(start 138.04132 86.04132)
-		(end 140 88)
-		(width 0.3)
-		(layer "F.Cu")
-		(net "+3V3")
-	)
-	(segment
-		(start 127.84868 103.61132)
-		(end 118.95868 112.50132)
-		(width 0.2)
-		(layer "B.Cu")
-		(net "+3V3")
-	)
-	(segment
-		(start 130.41132 103.61132)
-		(end 127.84868 103.61132)
-		(width 0.2)
-		(layer "B.Cu")
-		(net "+3V3")
-	)
-	(segment
-		(start 118.95868 112.50132)
-		(end 116.51132 112.50132)
-		(width 0.2)
-		(layer "B.Cu")
-		(net "+3V3")
-	)
-	(segment
 		(start 116.51132 102.34132)
 		(end 123.31132 102.34132)
@@
 	)
 	(segment
-		(start 111.96 88.58132)
-		(end 116.69132 88.58132)
-		(width 0.2)
-		(layer "B.Cu")
-		(net "OPENER_MOVING")
-	)
-	(segment
-		(start 116.69132 88.58132)
-		(end 120.55 92.44)
-		(width 0.2)
-		(layer "B.Cu")
-		(net "OPENER_MOVING")
-	)
-	(segment
-		(start 140 98.16)
-		(end 138.3 99.86)
-		(width 0.2)
-		(layer "B.Cu")
-		(net "OPENER_MOVING")
-	)
-	(segment
-		(start 129.97 99.64)
-		(end 134.33 104)
-		(width 0.2)
-		(layer "B.Cu")
-		(net "OPENER_MOVING")
-	)
-	(segment
-		(start 120.55 99.64)
-		(end 129.97 99.64)
-		(width 0.2)
-		(layer "B.Cu")
-		(net "OPENER_MOVING")
-	)
-	(segment
-		(start 138.3 99.86)
-		(end 138.3 104)
-		(width 0.2)
-		(layer "B.Cu")
-		(net "OPENER_MOVING")
-	)
-	(segment
-		(start 134.33 104)
-		(end 140 104)
-		(width 0.2)
-		(layer "B.Cu")
-		(net "OPENER_MOVING")
-	)
-	(segment
-		(start 120.55 92.44)
-		(end 120.55 99.64)
-		(width 0.2)
-		(layer "B.Cu")
-		(net "OPENER_MOVING")
-	)
-	(segment
 		(start 163.5 100.3)
 		(end 163.5 104.14)
@@
 		(net "Net-(R7-Pad2)")
 	)
+	(segment
+		(start 152.5 114.16)
+		(end 153.2 114.16)
+		(width 0.2)
+		(layer "B.Cu")
+		(net "/Opener control/LAMP")
+	)
+	(segment
+		(start 153.2 114.16)
+		(end 155.5 116.46)
+		(width 0.2)
+		(layer "B.Cu")
+		(net "/Opener control/LAMP")
+	)
+	(segment
+		(start 155.5 116.46)
+		(end 155.5 124.44)
+		(width 0.2)
+		(layer "B.Cu")
+		(net "/Opener control/LAMP")
+	)
 	(zone
