File: Circuit/GarageDoorController/opener-control.kicad_sch (KiCad schematic)
At the start: 17 parts, among them J4 JST PH 4-pin, U3 TLP222A, U4 PC817, U5 R-78E5.0-0.5, X1 Opener CON1

Commit message: Rev 2 PCB all references to FLASH changed LAMP + Controller housing
Connections:
- net FLASH renamed LAMP
Other:
- note added: "4-core cable from J4 (JST PH plug) to PB, GND, LAMP and +24."
- note added: "Check LAMP to GND with a meter while the door runs; if LAMP pulses, firmware treats pulses as moving."
- note added: "LAMP"
- note added: "OPENER_MOVING = XIAO D3 (GPIO5): LOW while the opener LAMP output is active (door moving)."
- note added: "R8 sets ~4.8 mA from a 24 V LAMP output (0.11 W). D4 protects the LED against reverse voltage."
- note removed: "4-core cable from J4 (JST PH plug) to PB, GND, FLASH and +24."
- note removed: "Check FLASH to GND with a meter while the door runs; if FLASH pulses, firmware treats pulses as moving."
- note removed: "FLASH"
- note removed: "OPENER_MOVING = XIAO D3 (GPIO5): LOW while the opener FLASH output is active (door moving)."
- note removed: "R8 sets ~4.8 mA from a 24 V FLASH output (0.11 W). D4 protects the LED against reverse voltage."
Changed lines of the file:
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@@
 		(title "Garage Door Controller - Opener Control")
 		(rev "2")
-		(comment 1 "PhotoMOS trigger to PB, optocoupler motion sense from FLASH")
+		(comment 1 "PhotoMOS trigger to PB, optocoupler motion sense from LAMP")
 	)
 	(polyline
@@
 		)
 	)
-	(text "R8 sets ~4.8 mA from a 24 V FLASH output (0.11 W). D4 protects the LED against reverse voltage."
+	(text "R8 sets ~4.8 mA from a 24 V LAMP output (0.11 W). D4 protects the LED against reverse voltage."
 		(exclude_from_sim no)
 		(at 30.48 142.24 0)
@@
 		)
 	)
-	(text "Check FLASH to GND with a meter while the door runs; if FLASH pulses, firmware treats pulses as moving."
+	(text "Check LAMP to GND with a meter while the door runs; if LAMP pulses, firmware treats pulses as moving."
 		(exclude_from_sim no)
 		(at 30.48 144.78 0)
@@
 		)
 	)
-	(text "FLASH"
+	(text "LAMP"
 		(exclude_from_sim no)
 		(at 224.79 86.96 0)
@@
 		)
 	)
-	(text "OPENER_MOVING = XIAO D3 (GPIO5): LOW while the opener FLASH output is active (door moving)."
+	(text "OPENER_MOVING = XIAO D3 (GPIO5): LOW while the opener LAMP output is active (door moving)."
 		(exclude_from_sim no)
 		(at 30.48 45.72 0)
@@
 		)
 	)
-	(text "4-core cable from J4 (JST PH plug) to PB, GND, FLASH and +24."
+	(text "4-core cable from J4 (JST PH plug) to PB, GND, LAMP and +24."
 		(exclude_from_sim no)
 		(at 191.77 111.76 0)
@@
 		)
 	)
-	(label "FLASH"
+	(label "LAMP"
 		(at 171.45 95.25 0)
 		(effects
@@
 		)
 	)
-	(label "FLASH"
+	(label "LAMP"
 		(at 208.28 86.36 180)
 		(effects
@@
 		)
 	)
-	(label "FLASH"
+	(label "LAMP"
 		(at 127 119.38 0)
 		(effects
